File: Power.kicad_sch (KiCad schematic)
At the start: 19 parts, among them U2 TPS563201DDCR, U3 TPS2116DRLR, U4 LMR54410DBVR

Commit message: fix: minor firmware issues
Parts:
- L2: symbol Device:L_Small -> Hardware Components:L_3u3_6A_Chilisin_MHCI06030-3R3M-S8
Changed lines of the file:
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@@
 	)
 	(symbol
-		(lib_id "Device:L_Small")
+		(lib_id "Hardware Components:L_3u3_6A_Chilisin_MHCI06030-3R3M-S8")
 		(at 170.18 40.64 90)
 		(unit 1)
